File: SYNOH052 carte etalon.kicad_sch (KiCad schematic)
At the start: 118 parts, among them J1 DIN41612_SYNOR, J10 Conn_02x08_Odd_Even, J11 Conn_02x08_Odd_Even, J12 Conn_02x08_Odd_Even, J13 Conn_02x08_Odd_Even, J14 Conn_02x08_Odd_Even, J15 Conn_02x08_Odd_Even, J16 Conn_02x08_Odd_Even, J17 Conn_02x08_Odd_Even, J18 Conn_01x0_P2.54mm_pinheader_v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, J19 Conn_01x0_P2.54mm_pinheader_v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, J2 Conn_01x32_P2.54mm_pinheader_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, J20 Conn_02x08_Odd_Even, J21 Conn_02x08_Odd_Even, J22 Conn_02x08_Odd_Even, J23 Conn_02x08_Odd_Even, J24 Conn_02x08_Odd_Even, J25 Conn_02x08_Odd_Even, J26 Conn_02x08_Odd_Even, J27 Conn_02x08_Odd_Even, J28 Conn_02x08_Odd_Even, J29 Conn_02x08_Odd_Even, J3 Conn_01x32_P2.54mm_pinheader_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, J30 Conn_02x08_Odd_Even, J31 Conn_02x08_Odd_Even, J32 Conn_01x0_P2.54mm_pinheader_v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, J33 Conn_01x0_P2.54mm_pinheader_v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, J34 Conn_01x0_P2.54mm_pinheader_v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, J35 Conn_01x0_P2.54mm_pinheader_v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, J36 Conn_01x0_P2.54mm_pinheader_v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, J37 Conn_01x0_P2.54mm_pinheader_v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, J38 Conn_01x0_P2.54mm_pinheader_v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, J39 Conn_01x0_P2.54mm_pinheader_v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, J4 Conn_02x08_Odd_Even, J40 Conn_01x0_P2.54mm_pinheader_v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, J41 Conn_01x0_P2.54mm_pinheader_v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, J42 Conn_01x0_P2.54mm_pinheader_v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, J43 Conn_01x0_P2.54mm_pinheader_v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, J44 Conn_01x0_P2.54mm_pinheader_v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, J45 Conn_01x0_P2.54mm_pinheader_v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, J46 Conn_01x0_P2.54mm_pinheader_v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, J47 Conn_01x0_P2.54mm_pinheader_v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, J48 Conn_01x0_P2.54mm_pinheader_v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, J49 Conn_01x0_P2.54mm_pinheader_v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, J5 Conn_02x08_Odd_Even, J50 Conn_01x0_P2.54mm_pinheader_v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, J51 Conn_01x0_P2.54mm_pinheader_v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, J52 Conn_01x0_P2.54mm_pinheader_v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, J53 Conn_01x0_P2.54mm_pinheader_v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, J54 Conn_01x0_P2.54mm_pinheader_v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, J55 Conn_01x0_P2.54mm_pinheader_v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, J56 Conn_01x0_P2.54mm_pinheader_v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, J57 Conn_01x0_P2.54mm_pinheader_v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, J58 Conn_01x0_P2.54mm_pinheader_v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, J59 Conn_01x0_P2.54mm_pinheader_v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, J6 Conn_02x08_Odd_Even, J60 Conn_01x0_P2.54mm_pinheader_v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, J61 Conn_01x0_P2.54mm_pinheader_v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, J62 Conn_01x0_P2.54mm_pinheader_v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, J63 Conn_01x0_P2.54mm_pinheader_v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, J64 Conn_01x0_P2.54mm_pinheader_v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, J65 Conn_01x0_P2.54mm_pinheader_v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, J66 Conn_01x0_P2.54mm_pinheader_v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, J67 Conn_01x0_P2.54mm_pinheader_v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, J68 Conn_01x0_P2.54mm_pinheader_v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, J69 Conn_01x0_P2.54mm_pinheader_v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, J7 Conn_02x08_Odd_Even, J70 Conn_01x0_P2.54mm_pinheader_v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, J71 Conn_01x0_P2.54mm_pinheader_v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, J72 Conn_01x0_P2.54mm_pinheader_v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, J73 Conn_01x0_P2.54mm_pinheader_v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, J74 Conn_01x0_P2.54mm_pinheader_v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, J75 Conn_01x0_P2.54mm_pinheader_v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, J76 Conn_01x0_P2.54mm_pinheader_v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, J77 Conn_01x0_P2.54mm_pinheader_v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, J78 Conn_01x0_P2.54mm_pinheader_v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, J79 Conn_01x0_P2.54mm_pinheader_v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, J8 Conn_02x08_Odd_Even, J80 Conn_01x0_P2.54mm_pinheader_v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, J81 Conn_01x0_P2.54mm_pinheader_v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

Commit message: version 21/03/2023 Signed-off-by: testbanc <banctest3@gmail.com>
Parts:
- C1: Distributeur 1 (none) -> 652-0083(RS); Fabreference (none) -> VJ0603A100JXBAC; Fabriquant (none) -> Vishay; now left out of the parts list
- C10: value 10000µ -> 10000u; Distributeur 1 (none) -> 711-1214(RS); Fabreference (none) -> RS PRO; Fabriquant (none) -> RS PRO
- C11, C12: Champ4 (none) -> Fabriquant; Champ5 (none) -> Fabreference; Champ6 (none) -> Omicron; Champ7 (none) -> Distributeur 1; Champ8 (none) -> Distributeur 2
- C2: Distributeur 1 (none) -> 205-3319(RS); Fabreference (none) -> C0603C101J3GACTU; Fabriquant (none) -> KEMET
- C3: Distributeur 1 (none) -> 272-7830(RS); Fabreference (none) -> VJ0603A102FXACW1BC; Fabriquant (none) -> Vishay
- C4: Distributeur 1 (none) -> 651-9998(RS); Fabreference (none) -> VJ1210A103FXAAT; Fabriquant (none) -> Vishay
- C5: Distributeur 1 (none) -> 272-7888(RS); Fabreference (none) -> VJ0603Y104KXBCW1BC; Fabriquant (none) -> Vishay
- C6: value 1µ -> 1u; Distributeur 1 (none) -> 272-7946(RS); Fabreference (none) -> VJ0805Y105KXATW1BC; Fabriquant (none) -> Vishay
- C7: value 10µ -> 10u; Distributeur 1 (none) -> 152-6096(RS); Fabreference (none) -> T356B105K050AT; Fabriquant (none) -> KEMET
- C8: value 100µ -> 100u; Distributeur 1 (none) -> 711-2096(RS); Fabreference (none) -> RS PRO; Fabriquant (none) -> RS PRO
- C9: value 1000µ -> 1000u; Distributeur 1 (none) -> 711-0842P(RS); Fabreference (none) -> RS PRO; Fabriquant (none) -> RS PRO
- J1: Distributeur 1 (none) -> RS:470-465; Distributeur 2 (none) -> F:1096940; Distributeur 3 (none) -> DK:1195-2891-ND; Distributeur1 RS:470-465 -> (none); Distributeur2 F:1096940 -> (none); Distributeur3 DK:1195-2891-ND -> (none)
- J10, J11, J12, J13, J14, J15, J16, J17, J20, J21, J22, J23, J24, J25, J26, J27, J28, J29, J30, J31, J4, J5, J6, J7, J8, J9: Distributeur 1 (none) -> F:2886108; Distributeur 2 (none) -> M:649-77313-118-72LF; Distributeur1 F:2886108 -> (none); Distributeur2 M:649-77313-118-72LF -> (none)
- J18, J19, J2, J3, J32, J33, J34, J35, J36, J37, J38, J39, J40, J41, J42, J43, J44, J45, J46, J47, J48, J49, J50, J51, J52, J53, J54, J55, J56, J57, J58, J59, J60, J61, J62, J63, J64, J65, J66, J67, J68, J69, J70, J71, J72, J73, J74, J75, J76, J77, J78, J79, J80, J81, J82, J83, J84, J85, J86, J87, J88, J89, J90, J91: Distributeur 1 (none) -> DK:609-6203-ND; Distributeur 2 (none) -> M:77311-102-36LF; Distributeur1 DK:609-6203-ND -> (none); Distributeur2 M:77311-102-36LF -> (none)
- R1: Distributeur 1 (none) -> 812-1821P; Fabreference (none) -> CRCW12061R00FKEAHP; Fabriquant (none) -> Vishay
- R10: Distributeur 1 (none) -> 819-8773(RS); Fabreference (none) -> CRHV2512AF500MFKET; Fabriquant (none) -> Vishay
- R2: Distributeur 1 (none) -> 788-8093 (RS); Fabreference (none) -> RLP0310R00FB15; Fabriquant (none) -> Vishay
- R3: Distributeur 1 (none) -> 880-2188 (Rs); Fabreference (none) -> RCP1206W100RGEB; Fabriquant (none) -> Vishay
- R4: Distributeur 1 (none) -> 679-1844(Rs); Fabreference (none) -> CRCW12061K00FKEA; Fabriquant (none) -> Vishay
- R5: Distributeur 1 (none) -> 218-2759 (RS); Fabreference (none) -> P2TC1206D1002LNTA; Fabriquant (none) -> Vishay
- R6: Distributeur 1 (none) -> 684-2645 (RS); Fabreference  (none) -> P1206C1003WNTA; Fabriquant (none) -> Vishay
- R7: Distributeur 1 (none) -> 684-2601(RS); Fabreference (none) -> P1206Y1004BNTA; Fabriquant (none) -> Vishay
- R8: Distributeur 1 (none) -> 819-8732P(RS); Fabreference (none) -> CRHV1206AF10M0FKET; Fabriquant (none) -> Vishay
- R9: Distributeur 1 (none) -> 819-8745P; Fabreference (none) -> CRHV1206AF100MFKET; Fabriquant (none) -> Vishay
